File: can_bus.kicad_sch (KiCad schematic)
At the start: 12 parts, among them P5 TERM, P6 TERM, U2 IFX1050GVIOXUMA1

Commit message: Schematic checked
Parts:
- removed C3: 100nF/50V, Capacitors_Smd_0603:100nF_0603, symbol Capacitors_Smd0603:100nF_0603
- added C1: 100nF/50V, Capacitors_Smd_0603:100nF_0603, symbol Capacitors_Smd0603:100n
- renumbered C4 to C2, D4 to D1, D5 to D2, D6 to D3, F3 to F1, F4 to F2, P5 to P3, P6 to P4, R3 to R1, R4 to R2, U2 to U1
Connections:
- net GND: now also C1.2
- net POWER_IN_5V0: now also C1.1
Changed lines of the file:
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@@
   (symbol (lib_id "Resistors_Smd0805:60.4R") (at 237.49 140.97 0)
     (in_bom yes) (on_board yes)
-    (property "Reference" "R3" (id 0) (at 231.5211 140.2091 0)
+    (property "Reference" "R1" (id 0) (at 231.5211 140.2091 0)
       (effects (font (size 1.27 1.27)) (justify left))
     )
@@
   (symbol (lib_id "Resistors_Smd0805:60.4R") (at 237.49 156.21 0)
     (in_bom yes) (on_board yes)
-    (property "Reference" "R4" (id 0) (at 231.5211 155.4491 0)
+    (property "Reference" "R2" (id 0) (at 231.5211 155.4491 0)
       (effects (font (size 1.27 1.27)) (justify left))
     )
@@
   (symbol (lib_id "Diodes:SMAJ18CA") (at 264.16 132.08 270)
     (in_bom yes) (on_board yes)
-    (property "Reference" "D4" (id 0) (at 266.7762 130.9116 90)
+    (property "Reference" "D1" (id 0) (at 266.7762 130.9116 90)
       (effects (font (size 1.27 1.27)) (justify left))
     )
@@
   (symbol (lib_id "Diodes:SMAJ18CA") (at 264.16 147.32 270)
     (in_bom yes) (on_board yes)
-    (property "Reference" "D5" (id 0) (at 266.7762 146.1516 90)
+    (property "Reference" "D2" (id 0) (at 266.7762 146.1516 90)
       (effects (font (size 1.27 1.27)) (justify left))
     )
@@
   (symbol (lib_id "Diodes:SMAJ18CA") (at 264.16 162.56 270)
     (in_bom yes) (on_board yes)
-    (property "Reference" "D6" (id 0) (at 266.7762 161.3916 90)
+    (property "Reference" "D3" (id 0) (at 266.7762 161.3916 90)
       (effects (font (size 1.27 1.27)) (justify left))
     )
@@
     (pin "2")
   )
-  (symbol (lib_id "Capacitors_Smd0603:100nF_0603") (at 180.34 128.27 0) (mirror x)
-    (in_bom yes) (on_board yes)
-    (property "Reference" "C3" (id 0) (at 177.0126 127.1016 0)
-      (effects (font (size 1.27 1.27)) (justify right))
-    )
-    (property "Value" "100nF/50V" (id 1) (at 177.0126 129.413 0)
-      (effects (font (size 1.27 1.27)) (justify right))
+  (symbol (lib_id "Capacitors_Smd0603:100n") (at 180.34 128.27 0)
+    (in_bom yes) (on_board yes)
+    (property "Reference" "C1" (id 0) (at 176.0475 124.9691 0)
+      (effects (font (size 1.27 1.27)) (justify left))
+    )
+    (property "Value" "100nF/50V" (id 1) (at 168.4275 131.0778 0)
+      (effects (font (size 1.27 1.27)) (justify left))
     )
     (property "Footprint" "Capacitors_Smd_0603:100nF_0603" (id 2) (at 180.34 128.27 0)
       (effects (font (size 1.524 1.524)) hide)
     )
-    (property "Datasheet" "Smd_0603/Components_Documentation/KEM_C1005_Y5V_SMD.pdf" (id 3) (at 183.6674 125.9586 0)
-      (effects (font (size 1.524 1.524)) (justify left) hide)
+    (property "Datasheet" "Capacitors/Smd_0603/Components_Documentation/KEM_C1005_Y5V_SMD.pdf" (id 3) (at 180.34 128.27 0)
+      (effects (font (size 1.524 1.524)) hide)
+    )
+    (property "Manufacturer" "SAMSUNG" (id 4) (at 180.34 128.27 0)
+      (effects (font (size 1.27 1.27)) hide)
+    )
+    (property "Manufacturer Part Number" "CL10B104JB8NNNC" (id 5) (at 180.34 128.27 0)
+      (effects (font (size 1.27 1.27)) hide)
+    )
+    (property "Supplier" "TME" (id 6) (at 180.34 128.27 0)
+      (effects (font (size 1.27 1.27)) hide)
+    )
+    (property "Supplier Part Number" "CL10B104JB8NNNC" (id 7) (at 180.34 128.27 0)
+      (effects (font (size 1.27 1.27)) hide)
+    )
+    (property "URL" "https://www.tme.eu/pl/details/cl10b104jb8nnnc/kondensatory-mlcc-smd-0603/samsung/" (id 8) (at 180.34 128.27 0)
+      (effects (font (size 1.27 1.27)) hide)
+    )
+    (property "Price@1pc" "0,04540" (id 9) (at 180.34 128.27 0)
+      (effects (font (size 1.27 1.27)) hide)
+    )
+    (property "Price@1000pcs" "0,02231" (id 10) (at 180.34 128.27 0)
+      (effects (font (size 1.27 1.27)) hide)
+    )
+    (property "Package" "0603" (id 11) (at 180.34 128.27 0)
+      (effects (font (size 1.27 1.27)) hide)
     )
     (pin "1")
@@
   (symbol (lib_id "Capacitors_Smd0603:100n") (at 245.11 148.59 90)
     (in_bom yes) (on_board yes)
-    (property "Reference" "C4" (id 0) (at 245.11 143.8614 90))
+    (property "Reference" "C2" (id 0) (at 245.11 143.8614 90))
     (property "Value" "100nF/50V" (id 1) (at 245.11 152.5101 90))
     (property "Footprint" "Capacitors_Smd_0603:100nF_0603" (id 2) (at 245.11 148.59 0)
@@
   (symbol (lib_id "Goldpin_2_54mm:GOLDPIN_2_2_54MM") (at 220.98 144.78 270)
     (in_bom yes) (on_board yes) (fields_autoplaced)
-    (property "Reference" "P5" (id 0) (at 224.1551 140.5269 90)
+    (property "Reference" "P3" (id 0) (at 224.1551 140.5269 90)
       (effects (font (size 1.524 1.524)) (justify left))
     )
@@
   (symbol (lib_id "Goldpin_2_54mm:GOLDPIN_2_2_54MM") (at 220.98 151.13 90)
     (in_bom yes) (on_board yes) (fields_autoplaced)
-    (property "Reference" "P6" (id 0) (at 224.1551 153.6079 90)
+    (property "Reference" "P4" (id 0) (at 224.1551 153.6079 90)
       (effects (font (size 1.524 1.524)) (justify right))
     )
@@
   (symbol (lib_id "Ptc_Smd_Fuses:SN005-60") (at 290.83 139.7 0)
     (in_bom yes) (on_board yes)
-    (property "Reference" "F3" (id 0) (at 290.83 132.9436 0))
+    (property "Reference" "F1" (id 0) (at 290.83 132.9436 0))
     (property "Value" "SN005-60" (id 1) (at 290.83 135.255 0))
     (property "Footprint" "Smd_Ptc_Fuses:SN005-60" (id 2) (at 290.83 139.7 0)
@@
   (symbol (lib_id "Ptc_Smd_Fuses:SN005-60") (at 290.83 154.94 0)
     (in_bom yes) (on_board yes)
-    (property "Reference" "F4" (id 0) (at 290.83 148.1836 0))
+    (property "Reference" "F2" (id 0) (at 290.83 148.1836 0))
     (property "Value" "SN005-60" (id 1) (at 290.83 150.495 0))
     (property "Footprint" "Smd_Ptc_Fuses:SN005-60" (id 2) (at 290.83 154.94 0)
@@
   (symbol (lib_id "Communication_Interfaces:IFX1050GVIOXUMA1") (at 190.5 149.86 0)
     (in_bom yes) (on_board yes)
-    (property "Reference" "U2" (id 0) (at 200.66 132.08 0))
+    (property "Reference" "U1" (id 0) (at 200.66 132.08 0))
     (property "Value" "IFX1050GVIOXUMA1" (id 1) (at 200.66 134.62 0))
     (property "Footprint" "Communication_Interfaces:IFX1050GVIOXUMA1" (id 2) (at 204.47 172.72 0)

Commit message: Finalized project
Parts:
- renumbered C1 to C3, C2 to C4, D1 to D4, D2 to D5, D3 to D6, F1 to F3, F2 to F4, P3 to P5, P4 to P6, R1 to R3, R2 to R4, U1 to U2
Changed lines of the file:
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@@
   (symbol (lib_id "Resistors_Smd0805:60.4R") (at 237.49 140.97 0)
     (in_bom yes) (on_board yes)
-    (property "Reference" "R1" (id 0) (at 231.5211 140.2091 0)
+    (property "Reference" "R3" (id 0) (at 231.5211 140.2091 0)
       (effects (font (size 1.27 1.27)) (justify left))
     )
@@
   (symbol (lib_id "Resistors_Smd0805:60.4R") (at 237.49 156.21 0)
     (in_bom yes) (on_board yes)
-    (property "Reference" "R2" (id 0) (at 231.5211 155.4491 0)
+    (property "Reference" "R4" (id 0) (at 231.5211 155.4491 0)
       (effects (font (size 1.27 1.27)) (justify left))
     )
@@
   (symbol (lib_id "Diodes:SMAJ18CA") (at 264.16 132.08 270)
     (in_bom yes) (on_board yes)
-    (property "Reference" "D1" (id 0) (at 266.7762 130.9116 90)
+    (property "Reference" "D4" (id 0) (at 266.7762 130.9116 90)
       (effects (font (size 1.27 1.27)) (justify left))
     )
@@
   (symbol (lib_id "Diodes:SMAJ18CA") (at 264.16 147.32 270)
     (in_bom yes) (on_board yes)
-    (property "Reference" "D2" (id 0) (at 266.7762 146.1516 90)
+    (property "Reference" "D5" (id 0) (at 266.7762 146.1516 90)
       (effects (font (size 1.27 1.27)) (justify left))
     )
@@
   (symbol (lib_id "Diodes:SMAJ18CA") (at 264.16 162.56 270)
     (in_bom yes) (on_board yes)
-    (property "Reference" "D3" (id 0) (at 266.7762 161.3916 90)
+    (property "Reference" "D6" (id 0) (at 266.7762 161.3916 90)
       (effects (font (size 1.27 1.27)) (justify left))
     )
@@
   (symbol (lib_id "Capacitors_Smd0603:100n") (at 180.34 128.27 0)
     (in_bom yes) (on_board yes)
-    (property "Reference" "C1" (id 0) (at 176.0475 124.9691 0)
+    (property "Reference" "C3" (id 0) (at 176.0475 124.9691 0)
       (effects (font (size 1.27 1.27)) (justify left))
     )
@@
   (symbol (lib_id "Capacitors_Smd0603:100n") (at 245.11 148.59 90)
     (in_bom yes) (on_board yes)
-    (property "Reference" "C2" (id 0) (at 245.11 143.8614 90))
+    (property "Reference" "C4" (id 0) (at 245.11 143.8614 90))
     (property "Value" "100nF/50V" (id 1) (at 245.11 152.5101 90))
     (property "Footprint" "Capacitors_Smd_0603:100nF_0603" (id 2) (at 245.11 148.59 0)
@@
   (symbol (lib_id "Goldpin_2_54mm:GOLDPIN_2_2_54MM") (at 220.98 144.78 270)
     (in_bom yes) (on_board yes) (fields_autoplaced)
-    (property "Reference" "P3" (id 0) (at 224.1551 140.5269 90)
+    (property "Reference" "P5" (id 0) (at 224.1551 140.5269 90)
       (effects (font (size 1.524 1.524)) (justify left))
     )
@@
   (symbol (lib_id "Goldpin_2_54mm:GOLDPIN_2_2_54MM") (at 220.98 151.13 90)
     (in_bom yes) (on_board yes) (fields_autoplaced)
-    (property "Reference" "P4" (id 0) (at 224.1551 153.6079 90)
+    (property "Reference" "P6" (id 0) (at 224.1551 153.6079 90)
       (effects (font (size 1.524 1.524)) (justify right))
     )
@@
   (symbol (lib_id "Ptc_Smd_Fuses:SN005-60") (at 290.83 139.7 0)
     (in_bom yes) (on_board yes)
-    (property "Reference" "F1" (id 0) (at 290.83 132.9436 0))
+    (property "Reference" "F3" (id 0) (at 290.83 132.9436 0))
     (property "Value" "SN005-60" (id 1) (at 290.83 135.255 0))
     (property "Footprint" "Smd_Ptc_Fuses:SN005-60" (id 2) (at 290.83 139.7 0)
@@
   (symbol (lib_id "Ptc_Smd_Fuses:SN005-60") (at 290.83 154.94 0)
     (in_bom yes) (on_board yes)
-    (property "Reference" "F2" (id 0) (at 290.83 148.1836 0))
+    (property "Reference" "F4" (id 0) (at 290.83 148.1836 0))
     (property "Value" "SN005-60" (id 1) (at 290.83 150.495 0))
     (property "Footprint" "Smd_Ptc_Fuses:SN005-60" (id 2) (at 290.83 154.94 0)
@@
   (symbol (lib_id "Communication_Interfaces:IFX1050GVIOXUMA1") (at 190.5 149.86 0)
     (in_bom yes) (on_board yes)
-    (property "Reference" "U1" (id 0) (at 200.66 132.08 0))
+    (property "Reference" "U2" (id 0) (at 200.66 132.08 0))
     (property "Value" "IFX1050GVIOXUMA1" (id 1) (at 200.66 134.62 0))
     (property "Footprint" "Communication_Interfaces:IFX1050GVIOXUMA1" (id 2) (at 204.47 172.72 0)

Commit message: Finalized project
Parts:
- removed D4, D5, D6: SMAJ18CA, Diodes:SMAJ18CA_SMD_DO214AC, symbol Diodes:SMAJ18CA
- added D2: PESD2CAN, ESD_Protectors:PESD2CAN.215, symbol esd_protectors:PESD2CAN
Connections:
- net GND: now also D2.3 (GND)
- net at F4.1, P6.1, U2.6 (CANL): now also D2.1 (I/O1)
- net at F3.1, P5.2, U2.7 (CANH): now also D2.2 (I/O2)
Other:
- moved on the sheet: F3, F4
