File: standalone_can_bus.kicad_sch (KiCad schematic)
At the start: 22 parts, among them P10 TERM, P11 TERM, U3 MCP2515, U4 MCP2551, X1 8MHZ

Commit message: Schematic checked
Parts:
- removed R5: 10k, Resistor_Smd_0603:10k_0603, symbol Resistors_Smd0603:10k_0603
- added R5: 10k, Resistor_Smd_0603:10k_0603, symbol Resistors_Smd0603:10k
- C5, C8, C9: symbol Capacitors_Smd0603:100nF_0603 -> Capacitors_Smd0603:100n
- R6, R7: symbol Resistors_Smd0603:47k_0603 -> Resistors_Smd0603:47k; Developer (none) -> MW; LCSC Part #(optional) (none) -> C105579; Manufacturer (none) -> Royal Ohm; Manufacturer Part Number (none) -> 0603SAF4702T5E; Price@1000pcs (none) -> 0,00813; Price@1pc (none) -> 0,03012; Supplier (none) -> Tme; Supplier Part Number (none) -> SMD0603-47K-1%; URL (none) -> https://www.tme.eu/pl/details/smd0603-47k-1%25/rezystory-sm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
- R8: symbol Resistors_Smd0603:100R_0603 -> Resistors_Smd0603:100R; Developer (none) -> MW; LCSC Part #(optional) (none) -> C269700; Manufacturer (none) -> Royal Ohm; Manufacturer Part Number (none) -> CQ03SAF1000T5E; Price@100pcs (none) -> 0,03414; Price@1pc (none) -> 0,07305; Supplier (none) -> Tme; Supplier Part Number (none) -> CQ0603-100R-1%; URL (none) -> https://www.tme.eu/pl/details/cq0603-100r-1%25/rezystory-sm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
Connections:
- net GND: now also U3.21 (EP)
- net POWER_VIN_3V3: now also R5.2
- net at C8.1, U3.17 (~RST): now also R5.1
Changed lines of the file:
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@@
+    (stroke (width 0) (type solid) (color 0 0 0 0))
+  )
+  (wire (pts (xy 124.46 184.15) (xy 124.46 185.42))
     (stroke (width 0) (type solid) (color 0 0 0 0))
   )
@@
   )
   (wire (pts (xy 264.16 137.16) (xy 284.48 137.16))
+    (stroke (width 0) (type solid) (color 0 0 0 0))
+  )
+  (wire (pts (xy 276.86 118.11) (xy 276.86 120.65))
     (stroke (width 0) (type solid) (color 0 0 0 0))
   )
@@
     (pin "1")
   )
-  (symbol (lib_id "power:GND") (at 281.94 128.27 90) (mirror x) (unit 1)
+  (symbol (lib_id "power:GND") (at 276.86 120.65 180) (unit 1)
+    (in_bom yes) (on_board yes)
+    (property "Reference" "#PWR0179" (id 0) (at 276.86 123.19 0)
+      (effects (font (size 0.762 0.762)) hide)
+    )
+    (property "Value" "GND" (id 1) (at 276.86 118.11 0)
+      (effects (font (size 0.762 0.762)) hide)
+    )
+    (property "Footprint" "" (id 2) (at 276.86 120.65 0)
+      (effects (font (size 1.524 1.524)))
+    )
+    (property "Datasheet" "" (id 3) (at 276.86 120.65 0)
+      (effects (font (size 1.524 1.524)))
+    )
+    (pin "1")
+  )
+  (symbol (lib_id "power:GND") (at 281.94 128.27 90) (unit 1)
     (in_bom yes) (on_board yes)
     (property "Reference" "#PWR0139" (id 0) (at 279.4 128.27 0)
@@
     (pin "1")
   )
-  (symbol (lib_id "Resistors_Smd0603:10k_0603") (at 199.39 143.51 90) (mirror x) (unit 1)
-    (in_bom yes) (on_board yes)
-    (property "Reference" "R5" (id 0) (at 199.39 140.97 90))
-    (property "Value" "10k" (id 1) (at 199.39 143.51 90))
+  (symbol (lib_id "Resistors_Smd0603:10k") (at 199.39 143.51 90) (unit 1)
+    (in_bom yes) (on_board yes) (fields_autoplaced)
+    (property "Reference" "R5" (id 0) (at 199.39 139.1878 90))
+    (property "Value" "10k" (id 1) (at 199.39 141.4865 90))
     (property "Footprint" "Resistor_Smd_0603:10k_0603" (id 2) (at 199.39 143.51 0)
       (effects (font (size 1.524 1.524)) hide)
@@
       (effects (font (size 1.27 1.27)) hide)
     )
-    (property "Manufacturer Part Number" "	0603SAJ0103T5E" (id 5) (at 199.39 143.51 0)
+    (property "Manufacturer Part Number" "0603SAJ0103T5E" (id 5) (at 199.39 143.51 0)
       (effects (font (size 1.27 1.27)) hide)
     )
@@
       (effects (font (size 1.27 1.27)) hide)
     )
-    (property "Developer" "WP" (id 11) (at 199.39 143.51 0)
+    (property "Developer" "MW" (id 11) (at 199.39 143.51 0)
       (effects (font (size 1.27 1.27)) hide)
     )
@@
     (pin "2")
   )
-  (symbol (lib_id "Resistors_Smd0603:47k_0603") (at 224.79 151.13 0) (mirror y) (unit 1)
+  (symbol (lib_id "Resistors_Smd0603:47k") (at 224.79 151.13 0) (mirror y) (unit 1)
     (in_bom yes) (on_board yes)
     (property "Reference" "R6" (id 0) (at 223.0628 149.9616 0)
@@
       (effects (font (size 1.524 1.524)) hide)
     )
-    (property "Datasheet" "Resistors/Smd_0603/Components_Documentation/Vishay_Resistors_SM0603.pdf" (id 3) (at 224.79 151.13 0)
+    (property "Datasheet" "https://www.tme.eu/Document/b315665a56acbc42df513c99b390ad98/ROYALOHM-THICKFILM.pdf" (id 3) (at 224.79 151.13 0)
       (effects (font (size 1.524 1.524)) hide)
     )
@@
       (effects (font (size 1.27 1.27)) hide)
     )
-    (pin "1")
-    (pin "2")
-  )
-  (symbol (lib_id "Resistors_Smd0603:47k_0603") (at 224.79 166.37 0) (mirror y) (unit 1)
+    (property "Manufacturer" "Royal Ohm" (id 5) (at 224.79 151.13 0)
+      (effects (font (size 1.27 1.27)) hide)
+    )
+    (property "Manufacturer Part Number" "0603SAF4702T5E" (id 6) (at 224.79 151.13 0)
+      (effects (font (size 1.27 1.27)) hide)
+    )
+    (property "Supplier" "Tme" (id 7) (at 224.79 151.13 0)
+      (effects (font (size 1.27 1.27)) hide)
+    )
+    (property "Supplier Part Number" "SMD0603-47K-1%" (id 8) (at 224.79 151.13 0)
+      (effects (font (size 1.27 1.27)) hide)
+    )
+    (property "URL" "https://www.tme.eu/pl/details/smd0603-47k-1%25/rezystory-smd-0603/royal-ohm/0603saf4702t5e/" (id 9) (at 224.79 151.13 0)
+      (effects (font (size 1.27 1.27)) hide)
+    )
+    (property "Price@1pc" "0,03012" (id 10) (at 224.79 151.13 0)
+      (effects (font (size 1.27 1.27)) hide)
+    )
+    (property "Price@1000pcs" "0,00813" (id 11) (at 224.79 151.13 0)
+      (effects (font (size 1.27 1.27)) hide)
+    )
+    (property "Developer" "MW" (id 12) (at 224.79 151.13 0)
+      (effects (font (size 1.27 1.27)) hide)
+    )
+    (property "LCSC Part #(optional)" "C105579" (id 13) (at 224.79 151.13 0)
+      (effects (font (size 1.27 1.27)) hide)
+    )
+    (pin "1")
+    (pin "2")
+  )
+  (symbol (lib_id "Resistors_Smd0603:47k") (at 224.79 166.37 0) (mirror y) (unit 1)
     (in_bom yes) (on_board yes)
     (property "Reference" "R7" (id 0) (at 223.0628 165.2016 0)
@@
       (effects (font (size 1.524 1.524)) hide)
     )
-    (property "Datasheet" "Resistors/Smd_0603/Components_Documentation/Vishay_Resistors_SM0603.pdf" (id 3) (at 224.79 166.37 0)
+    (property "Datasheet" "https://www.tme.eu/Document/b315665a56acbc42df513c99b390ad98/ROYALOHM-THICKFILM.pdf" (id 3) (at 224.79 166.37 0)
       (effects (font (size 1.524 1.524)) hide)
     )
@@
       (effects (font (size 1.27 1.27)) hide)
     )
-    (pin "1")
-    (pin "2")
-  )
-  (symbol (lib_id "Resistors_Smd0603:100R_0603") (at 273.05 128.27 90) (mirror x) (unit 1)
+    (property "Manufacturer" "Royal Ohm" (id 5) (at 224.79 166.37 0)
+      (effects (font (size 1.27 1.27)) hide)
+    )
+    (property "Manufacturer Part Number" "0603SAF4702T5E" (id 6) (at 224.79 166.37 0)
+      (effects (font (size 1.27 1.27)) hide)
+    )
+    (property "Supplier" "Tme" (id 7) (at 224.79 166.37 0)
+      (effects (font (size 1.27 1.27)) hide)
+    )
+    (property "Supplier Part Number" "SMD0603-47K-1%" (id 8) (at 224.79 166.37 0)
+      (effects (font (size 1.27 1.27)) hide)
+    )
+    (property "URL" "https://www.tme.eu/pl/details/smd0603-47k-1%25/rezystory-smd-0603/royal-ohm/0603saf4702t5e/" (id 9) (at 224.79 166.37 0)
+      (effects (font (size 1.27 1.27)) hide)
+    )
+    (property "Price@1pc" "0,03012" (id 10) (at 224.79 166.37 0)
+      (effects (font (size 1.27 1.27)) hide)
+    )
+    (property "Price@1000pcs" "0,00813" (id 11) (at 224.79 166.37 0)
+      (effects (font (size 1.27 1.27)) hide)
+    )
+    (property "Developer" "MW" (id 12) (at 224.79 166.37 0)
+      (effects (font (size 1.27 1.27)) hide)
+    )
+    (property "LCSC Part #(optional)" "C105579" (id 13) (at 224.79 166.37 0)
+      (effects (font (size 1.27 1.27)) hide)
+    )
+    (pin "1")
+    (pin "2")
+  )
+  (symbol (lib_id "Resistors_Smd0603:100R") (at 273.05 128.27 90) (mirror x) (unit 1)
     (in_bom yes) (on_board yes)
     (property "Reference" "R8" (id 0) (at 273.05 125.73 90))
@@
       (effects (font (size 1.524 1.524)) hide)
     )
-    (property "Datasheet" "Resistors/Smd_0603/Components_Documentation/Vishay_Resistors_SM0603.pdf" (id 3) (at 273.05 128.27 0)
+    (property "Datasheet" "https://www.tme.eu/Document/ec37243ca557adb02ebafc5c1ab83104/CQ%20datasheet.pdf" (id 3) (at 273.05 128.27 0)
       (effects (font (size 1.524 1.524)) hide)
     )
     (property "Package" "0603" (id 4) (at 273.05 128.27 0)
+      (effects (font (size 1.27 1.27)) hide)
+    )
+    (property "Manufacturer" "Royal Ohm" (id 5) (at 273.05 128.27 0)
+      (effects (font (size 1.27 1.27)) hide)
+    )
+    (property "Manufacturer Part Number" "CQ03SAF1000T5E" (id 6) (at 273.05 128.27 0)
+      (effects (font (size 1.27 1.27)) hide)
+    )
+    (property "Supplier" "Tme" (id 7) (at 273.05 128.27 0)
+      (effects (font (size 1.27 1.27)) hide)
+    )
+    (property "Supplier Part Number" "CQ0603-100R-1%" (id 8) (at 273.05 128.27 0)
+      (effects (font (size 1.27 1.27)) hide)
+    )
+    (property "URL" "https://www.tme.eu/pl/details/cq0603-100r-1%25/rezystory-smd-0603/royal-ohm/cq03saf1000t5e/" (id 9) (at 273.05 128.27 0)
+      (effects (font (size 1.27 1.27)) hide)
+    )
+    (property "Price@1pc" "0,07305" (id 10) (at 273.05 128.27 0)
+      (effects (font (size 1.27 1.27)) hide)
+    )
+    (property "Price@100pcs" "0,03414" (id 11) (at 273.05 128.27 0)
+      (effects (font (size 1.27 1.27)) hide)
+    )
+    (property "Developer" "MW" (id 12) (at 273.05 128.27 0)
+      (effects (font (size 1.27 1.27)) hide)
+    )
+    (property "LCSC Part #(optional)" "C269700" (id 13) (at 273.05 128.27 0)
       (effects (font (size 1.27 1.27)) hide)
     )
@@
     (pin "1")
   )
+  (symbol (lib_id "power:PWR_FLAG") (at 276.86 118.11 0) (unit 1)
+    (in_bom yes) (on_board yes) (fields_autoplaced)
+    (property "Reference" "#FLG0107" (id 0) (at 276.86 111.252 0)
+      (effects (font (size 0.762 0.762)) hide)
+    )
+    (property "Value" "PWR_FLAG" (id 1) (at 276.86 112.1207 0)
+      (effects (font (size 0.762 0.762)))
+    )
+    (property "Footprint" "" (id 2) (at 276.86 118.11 0)
+      (effects (font (size 1.524 1.524)))
+    )
+    (property "Datasheet" "" (id 3) (at 276.86 118.11 0)
+      (effects (font (size 1.524 1.524)))
+    )
+    (pin "1")
+  )
   (symbol (lib_id "Diodes:SMAJ18CA") (at 335.28 118.11 270) (unit 1)
     (in_bom yes) (on_board yes)
@@
     (pin "2")
   )
-  (symbol (lib_id "Capacitors_Smd0603:100nF_0603") (at 121.92 115.57 0) (mirror y) (unit 1)
+  (symbol (lib_id "Capacitors_Smd0603:100n") (at 121.92 115.57 0) (mirror y) (unit 1)
     (in_bom yes) (on_board yes)
     (property "Reference" "C5" (id 0) (at 118.5926 114.4016 0)
@@
     (pin "2")
   )
-  (symbol (lib_id "Capacitors_Smd0603:100nF_0603") (at 185.42 154.94 0) (mirror y) (unit 1)
+  (symbol (lib_id "Capacitors_Smd0603:100n") (at 185.42 154.94 0) (mirror y) (unit 1)
     (in_bom yes) (on_board yes)
     (property "Reference" "C8" (id 0) (at 182.0926 153.7716 0)
@@
     (pin "2")
   )
-  (symbol (lib_id "Capacitors_Smd0603:100nF_0603") (at 255.27 113.03 0) (unit 1)
+  (symbol (lib_id "Capacitors_Smd0603:100n") (at 255.27 113.03 0) (unit 1)
     (in_bom yes) (on_board yes)
     (property "Reference" "C9" (id 0) (at 258.5974 111.8616 0)

Commit message: Finalized project
Parts:
- removed R6, R7: 47k, Resistor_Smd_0603:47k_0603, symbol Resistors_Smd0603:47k
- removed U3: MCP2515, Communication_Interfaces:MCP2515-I-QFN20, symbol Communication_Interfaces:MCP2515
- added C14, C17, C18: 100nF/50V, Capacitors_Smd_0603:100nF_0603, symbol Capacitors_Smd0603:100n
- added C15, C16: 30pF/50V, Capacitors_Smd_0603:30pF_0603, symbol Capacitors_Smd0603:30pF_0603
- added D16, D17, D18: SMAJ18CA, Diodes:SMAJ18CA_SMD_DO214AC, symbol Diodes:SMAJ18CA
- added F10, F9: SN005-60, Smd_Ptc_Fuses:SN005-60, symbol Ptc_Smd_Fuses:SN005-60
- added R24, R27: 100R, Resistor_Smd_0603:100R_0603, symbol Resistors_Smd0603:100R
- added R25, R26: 60.4R, Resistor_Smd_0805:60.4R_0805, symbol Resistors_Smd0805:60.4R
- added U3: MCP2515_TSSOP20, Communication_Interfaces:MCP2515-I-TSSOP20, symbol Communication_Interfaces:MCP2515_TSSOP20
- added U8: MCP2512_VDFN14, Communication_Interfaces:MCP2512_VDFN14, symbol Communication_Interfaces:MCP2512_VDFN14
- added U9: MCP2551, Communication_Interfaces:MCP2551_SO8, symbol Communication_Interfaces:MCP2551
- added X2: 8MHZ, Resonators:ABM3AIG-8.000MHZ-8-1R-T, symbol Resonators:ABM3AIG-8.000MHZ-8-1R-T
Connections:
- net CAN_MISO: now also R27.1, U3.17 (SO)
- net CAN_MOSI: now also U3.16 (SI), U8.11 (SI)
- net CAN_SCK: now also U3.14 (SCK), U8.10 (SCK)
- net GND: now also C14.2, C15.2, C16.2, C17.2, C18.2, D16.1 (A), D18.2 (K), R24.2, U3.10 (GND), U8.7 (GND), U8.EP, U9.2 (VSS)
- net POWER_VIN_3V3: now also U4.5 (VREF), C14.1, U3.20 (VDD), U8.14 (VDD), U9.5 (VREF); no longer C9.1, U4.3 (VDD)
- net at U4.1 (TXD): now also U3.1 (TXCAN)
- net at U4.4 (RXD): now also U3.2 (RXCAN)
- net at C8.1, R5.1: now also U3.19 (~RST)
- net at C6.1, X1.1: now also U3.8 (OSC2)
- net at C7.1, X1.2: now also U3.9 (OSC1)
- net CAN_H renamed CAN_H0
- net CAN_L renamed CAN_L0
- new net: C16.1, U8.6 (OSC1), X2.2
- new net: C18.1, R25.2, R26.1
- new net: D17.2 (K), D18.1 (A), F10.1, R26.2, U9.6 (CANL)
- new net: D16.2 (K), D17.1 (A), F9.1, R25.1, U9.7 (CANH)
- new net: R27.2, U8.12 (SO)
- new net: C15.1, U8.5 (OSC2), X2.1
- new net: R24.1, U9.8 (RS)
- new net: U8.1 (TXCAN), U9.1 (TXD)
- new net: U8.2 (RXCAN), U9.4 (RXD)
- new net CAN_H1: F9.2
- new net CAN_L1: F10.2
- new net CAN_~CS0~: U3.18 (~CS)
- new net CAN_~CS1~: U8.13 (~CS)
- new net CAN_~INT0~: U3.13 (~INT)
- new net CAN_~INT1~: U8.4 (~INT)
- new net POWER_VIN_5V0: C17.1, C9.1, U4.3 (VDD), U9.3 (VDD)
- no-connect marks 6 -> 9
Other:
- moved on the sheet: C10, C5, C6, C7, C8, C9, D7, D8, D9, F5, F6, P10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

Commit message: Finalized project
Parts:
- removed D16, D17, D18, D7, D8, D9: SMAJ18CA, Diodes:SMAJ18CA_SMD_DO214AC, symbol Diodes:SMAJ18CA
- added D3, D4: PESD2CAN, ESD_Protectors:PESD2CAN.215, symbol esd_protectors:PESD2CAN
Connections:
- net GND: now also D3.3 (GND), D4.3 (GND)
- net at F5.1, P10.2, U4.7 (CANH): now also D3.2 (I/O2)
- net at F10.1, R26.2, U9.6 (CANL): now also D4.1 (I/O1)
- net at F6.1, P11.1, U4.6 (CANL): now also D3.1 (I/O1)
- net at F9.1, R25.1, U9.7 (CANH): now also D4.2 (I/O2)
Other:
- moved on the sheet: C18, F5, F6, R25, R26
